Commit message: auto save

File: src/roarm/urdf/roarm.urdf (robot description, URDF)
Before this commit: robot physics, 11 links, 10 joints
Joints:
- joint L4_to_L5_1_A: limit lower=-1.57 upper=0 effort=1000.0 velocity=0.5 -> lower=-2 upper=0 effort=1000.0 velocity=0.5
- joint L4_to_L5_1_B: limit lower=-1.57 upper=1.57 effort=1000.0 velocity=0.5 -> lower=-2 upper=1.57 effort=1000.0 velocity=0.5
- joint L4_to_L5_2_A: limit lower=-1.57 upper=1.57 effort=1000.0 velocity=0.5 -> lower=-2 upper=1.57 effort=1000.0 velocity=0.5
- joint L4_to_L5_2_B: limit lower=-1.57 upper=1.57 effort=1000.0 velocity=0.5 -> lower=-2 upper=1.57 effort=1000.0 velocity=0.5
- joint L5_1_A_to_L5_3_A: limit lower=-1.57 upper=0 effort=1000.0 velocity=0.5 -> lower=-2 upper=0 effort=1000.0 velocity=0.5
- joint L5_1_B_to_L5_3_B: limit lower=-1.57 upper=0 effort=1000.0 velocity=0.5 -> lower=-2 upper=0 effort=1000.0 velocity=0.5

Commit message: :poop:

File: src/roarm/urdf/roarm.urdf (robot description, URDF)
Before this commit: robot physics, 11 links, 10 joints
Links:
- added link r1_link; visual mesh filename=package://roarm/meshes/L1.stl
- added link r2_link; visual mesh filename=package://roarm/meshes/L2.stl
- added link r3_link; visual mesh filename=package://roarm/meshes/L3.stl
- added link r4_link; visual mesh filename=package://roarm/meshes/L4.stl
Joints:
- added joint R1_to_R2: type revolute, parent r1_link, child r2_link, origin xyz=0 0.041051 0.0534, axis 1 0 0, limit lower=-1.0467 upper=1.0467 effort=1000.0 velocity=0.5
- added joint R2_to_R3: type revolute, parent r2_link, child r3_link, origin xyz=0 0.119401 0.119401, axis 1 0 0, limit lower=-2.7 upper=2.7 effort=1000.0 velocity=0.5
- added joint R3_to_R4: type revolute, parent r3_link, child r4_link, origin xyz=0 0.090485 0.090455, axis 1 0 0, limit lower=-2.1 upper=2.1 effort=1000.0 velocity=0.5
- added joint base_to_R1: type revolute, parent base_link, child r1_link, origin xyz=0 -0.35 0.062, axis 0 0 1, limit lower=-3.14 upper=3.14 effort=1000.0 velocity=0.5
